Commit message: feat(sim): SO-101 손목 카메라 홀더(Hex-Nut Mount) gripper 부착
SO-ARM101 Hex-Nut Recess Wrist Camera Mount(32x32 UVC) 홀더를
gripper_link 에 고정 부착. 6D pose 는 STEP CAD 나사구멍 매칭으로 도출.

- 홀더 M3 2구멍(R1.65, 간격 8.1mm) <-> wrist_roll_follower hex-nut
  나사쌍(R1.6, 간격 8.1mm) 간격 정확 일치로 쌍 확정. 접촉면 밀착
  (홀더 x=0 <-> follower 외측 y=-24.22mm). STL 은 프린트 방향이라
  STEP CIRCLE 엔티티 파싱으로 정확 추출.
- transform(gripper_link 기준): xyz=-0.015 0.0240018 -0.0315503,
  rpy=-pi/2 0 -pi/2. 튜닝된 WristCamera(+y0.045)와 교차검증.

파일:
- urdf/assets/wrist_cam_mount_so101_v1.stl (mm 원본)
- so_arm101.urdf: wrist_cam_mount_link + fixed joint(scale 0.001)
- wrist_cam_mount.usd: STL->UsdGeom.Mesh (visual-only)
- so101_follower.usd: /so101_new_calib/gripper/WristCamMount reference

URDF 소비처=RMPFlow/cuMotion(xrdf gen)/MoveIt PATH E/FK ref. 시뮬
렌더는 별도 USD 라 둘 다 편집. cuMotion xrdf collision sphere 는 제외.
최종 시각확인은 Windows GUI(teleop_se3_agent.py --tune_cameras).

File: assets/robots/urdf/so_arm101.urdf (robot description, URDF)
Before this commit: robot so101_new_calib, 8 links, 7 joints
Links:
- added link wrist_cam_mount_link, mass 0.015; collision mesh filename=assets/wrist_cam_mount_so101_v1.stl scale=0.001 0.001 0.001; visual mesh filename=assets/wrist_cam_mount_so101_v1.stl scale=0.001 0.001 0.001
Joints:
- added joint wrist_cam_mount_joint: type fixed, parent gripper_link, child wrist_cam_mount_link, origin xyz=-0.015 0.0240018 -0.0315503 rpy=-1.5707963 0 -1.5707963, axis 0 0 0

Commit message: feat(sim): 손목/전면 카메라 홀더 사진기반 재설계 + 카메라 pose·home 정합
실물 사진(docs/pics/cube_desk) 기준으로 SO-101 손목/전면(belly) 카메라
홀더를 procedural 로 재제작하고, sim 카메라 pose·SM home 자세를 정합.

홀더 (scripts/assets/build_cam_holders.py 가 부모 링크 프레임[m]에 생성):
- wrist: 나사판 → 직각 얇은 융기 → 45° 숙인 enclosure(카메라 감쌈, 렌즈
  주둥이만 노출). gripper_link 의 hex-nut 나사쌍 결합.
- belly(front): 좁은 네모 기둥 → 넓고 얇은 backing 판(카메라 크기) → UVC
  카메라 노출. shoulder_link 앞면 장착(shoulder_pan 따라감).
- 카메라 목업 = UVC(렌즈 원통 + PCB 네모판), 양쪽 동일. holder=보라
  (material_a_3d_printed), 카메라=검정(material_black 신규).
- generic hex-nut STL/USD(wrist_cam_mount*) 폐기.

정합:
- pick_cube_env_cfg: _FRONT_CAM_LOCAL_POS (0.05)→(-0.083,0,0) — 새 belly
  홀더 렌즈 위치, observation.front 와 일치.
- pick_cube_state_machine: HOME_Q wrist_roll +90°→-90°(손목 카메라 마운트
  위로). _init_pose roll init 도 -90° 로 맞춰 grasp 시작 wrist 스윙 제거.

teleop_se3_agent: --public_ip 추가(PUBLIC_IP env + livestream mode 1 승격),
SM 과 동일 패턴. 원격 WebRTC livestream 관전용.

URDF/USD/env_cfg/teleop 의 front cam 은 동일 prim(/Robot/shoulder/FrontCamera).

File: assets/robots/urdf/so_arm101.urdf (robot description, URDF)
Before this commit: robot so101_new_calib, 9 links, 8 joints
Links:
- added link front_cam_mount_link, mass 0.020; collision mesh filename=assets/front_cam_holder_so101.stl; visual mesh filename=assets/front_cam_holder_so101.stl
- link wrist_cam_mount_link: geometry collision mesh filename=assets/wrist_cam_holder_so101.stl; visual mesh filename=assets/wrist_cam_holder_so101.stl
Joints:
- added joint front_cam_mount_joint: type fixed, parent shoulder_link, child front_cam_mount_link, origin xyz=0 0 0 rpy=0 0 0, axis 0 0 0
- joint wrist_cam_mount_joint: origin xyz=-0.015 0.0240018 -0.0315503 rpy=-1.5707963 0 -1.5707963 -> xyz=0 0 0 rpy=0 0 0
